File: Hardware/Top/RocketWatch-TOP.sch (EAGLE design)
At the start: 52 parts, among them SW1 SWITCH.MOM, SW2 SWITCH.MOM, SW5 SWITCH.MOM, U2 NRF52832_MODULE_MDBT42, U4 PCF8523

Commit message: finished top schematic and  board according to take 001 video
Parts:
- removed SW2, SW5: SWITCH.MOM, LinnesLab-Switches:SWITCH.MOM
- added SW6: SWITCH.MOM, LinnesLab-Switches:SWITCH.MOM
Connections:
- removed net VBATT: U4.VBAT
- new net SW1: SW1.1, SW6.1
- net GND: now also SW1.3, SW1.4, SW6.3, SW6.4, USB2.SHIELD
Other:
- note added: "PINS THAT NEED ASSIGNED DIGITAL OUTPUTS Digital GPIO CS.OLED RESET.OLED DC.OLED [SPI] [I2C] SD.CS (Optional) Card Detect1 and 2 DIGITAL INPUTS 3x Buttons Charge Status ANALOG INPUTS Battery Monitor ANALOG OUTPUTS"
- moved on the sheet: SW1
Changed lines of the file:
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@@
 </part>
 <part name="SW1" library="LinnesLab-Switches" deviceset="SWITCH.MOM" device=""/>
-<part name="SW2" library="LinnesLab-Switches" deviceset="SWITCH.MOM" device=""/>
-<part name="SW5" library="LinnesLab-Switches" deviceset="SWITCH.MOM" device=""/>
+<part name="GND1" library="LinnesLab-Symbols" deviceset="GND" device=""/>
+<part name="SW6" library="LinnesLab-Switches" deviceset="SWITCH.MOM" device=""/>
+<part name="GND3" library="LinnesLab-Symbols" deviceset="GND" device=""/>
 </parts>
 <sheets>
@@
 battery
 if desired</text>
-<text x="71.12" y="152.4" size="6.4516" layer="91" font="vector">nRF52832 Module</text>
-<text x="370.84" y="27.94" size="6.4516" layer="91" font="vector">Buttons</text>
-<text x="71.12" y="-7.62" size="6.4516" layer="91" font="vector">Power Management</text>
-<text x="223.52" y="5.08" size="6.4516" layer="91" font="vector">SD Card</text>
-<text x="355.6" y="-22.86" size="6.4516" layer="91" font="vector">Real-Time Clock</text>
-<text x="248.92" y="144.78" size="6.4516" layer="91" font="vector">Cortex Debugger/
+<text x="71.12" y="152.4" size="6.4516" layer="97" font="vector">nRF52832 Module</text>
+<text x="370.84" y="27.94" size="6.4516" layer="97" font="vector">Buttons</text>
+<text x="71.12" y="-7.62" size="6.4516" layer="97" font="vector">Power Management</text>
+<text x="223.52" y="5.08" size="6.4516" layer="97" font="vector">SD Card</text>
+<text x="355.6" y="-22.86" size="6.4516" layer="97" font="vector">Real-Time Clock</text>
+<text x="248.92" y="144.78" size="6.4516" layer="97" font="vector">Cortex Debugger/
 Programmer</text>
 <text x="269.24" y="86.36" size="6.4516" layer="91" font="vector">RTC
 </text>
-<text x="383.54" y="162.56" size="6.4516" layer="91" font="vector">OLED</text>
+<text x="383.54" y="162.56" size="6.4516" layer="97" font="vector">OLED</text>
 <wire x1="-50.8" y1="190.5" x2="449.58" y2="190.5" width="0.254" layer="94"/>
 <wire x1="449.58" y1="190.5" x2="449.58" y2="-111.76" width="0.254" layer="94"/>
 <wire x1="449.58" y1="-111.76" x2="-50.8" y2="-111.76" width="0.254" layer="94"/>
 <wire x1="-50.8" y1="-111.76" x2="-50.8" y2="190.5" width="0.254" layer="94"/>
-<wire x1="-40.64" y1="185.42" x2="441.96" y2="185.42" width="0.254" layer="94" style="longdash"/>
+<wire x1="-43.18" y1="185.42" x2="441.96" y2="185.42" width="0.254" layer="94" style="longdash"/>
 <wire x1="441.96" y1="185.42" x2="441.96" y2="-106.68" width="0.254" layer="94" style="longdash"/>
 <wire x1="441.96" y1="-106.68" x2="-43.18" y2="-106.68" width="0.254" layer="94" style="longdash"/>
 <wire x1="-43.18" y1="-106.68" x2="-43.18" y2="185.42" width="0.254" layer="94" style="longdash"/>
-<wire x1="-43.18" y1="185.42" x2="-40.64" y2="185.42" width="0.254" layer="94" style="longdash"/>
 <wire x1="-43.18" y1="5.08" x2="218.44" y2="5.08" width="0.254" layer="97" style="longdash"/>
 <wire x1="218.44" y1="5.08" x2="218.44" y2="45.72" width="0.254" layer="97" style="longdash"/>
@@
 <wire x1="314.96" y1="-7.62" x2="314.96" y2="-106.68" width="0.254" layer="97" style="longdash"/>
 <wire x1="200.66" y1="2.54" x2="200.66" y2="-104.14" width="0.254" layer="97" style="longdash"/>
+<text x="-101.6" y="119.38" size="1.778" layer="97">PINS THAT NEED ASSIGNED
+DIGITAL OUTPUTS
+Digital GPIO
+CS.OLED
+RESET.OLED
+DC.OLED
+[SPI]
+[I2C]
+SD.CS
+(Optional) Card Detect1 and 2
+DIGITAL INPUTS
+3x Buttons
+Charge Status
+ANALOG INPUTS
+Battery Monitor
+ANALOG OUTPUTS</text>
 </plain>
 <instances>
@@
 <attribute name="MFN_MANUFACTURER" x="373.38" y="-50.8" size="1.27" layer="96" display="off"/>
 </instance>
-<instance part="SW1" gate="G$1" x="355.6" y="7.62" smashed="yes">
-<attribute name="NAME" x="355.6" y="12.446" size="1.778" layer="95" font="vector" align="bottom-center"/>
-<attribute name="VALUE" x="355.6" y="4.826" size="1.778" layer="96" font="vector" align="top-center"/>
-</instance>
-<instance part="SW2" gate="G$1" x="383.54" y="7.62" smashed="yes">
-<attribute name="NAME" x="383.54" y="12.446" size="1.778" layer="95" font="vector" align="bottom-center"/>
-<attribute name="VALUE" x="383.54" y="4.826" size="1.778" layer="96" font="vector" align="top-center"/>
-</instance>
-<instance part="SW5" gate="G$1" x="411.48" y="7.62" smashed="yes">
-<attribute name="NAME" x="411.48" y="12.446" size="1.778" layer="95" font="vector" align="bottom-center"/>
-<attribute name="VALUE" x="411.48" y="4.826" size="1.778" layer="96" font="vector" align="top-center"/>
+<instance part="SW1" gate="G$1" x="350.52" y="12.7" smashed="yes">
+<attribute name="NAME" x="350.52" y="17.526" size="1.778" layer="95" font="vector" align="bottom-center"/>
+<attribute name="VALUE" x="350.52" y="9.906" size="1.778" layer="96" font="vector" align="top-center"/>
+</instance>
+<instance part="GND1" gate="G$1" x="360.68" y="5.08" smashed="yes">
+<attribute name="VALUE" x="360.68" y="4.826" size="1.778" layer="96" align="top-center"/>
+</instance>
+<instance part="SW6" gate="G$1" x="386.08" y="12.7" smashed="yes">
+<attribute name="NAME" x="386.08" y="17.526" size="1.778" layer="95" font="vector" align="bottom-center"/>
+<attribute name="VALUE" x="386.08" y="9.906" size="1.778" layer="96" font="vector" align="top-center"/>
+</instance>
+<instance part="GND3" gate="G$1" x="396.24" y="5.08" smashed="yes">
+<attribute name="VALUE" x="396.24" y="4.826" size="1.778" layer="96" align="top-center"/>
 </instance>
 </instances>
@@
 <pinref part="GND40" gate="G$1" pin="GND"/>
 <wire x1="58.42" y1="-66.04" x2="58.42" y2="-73.66" width="0.1524" layer="91"/>
+<pinref part="USB2" gate="G$1" pin="SHIELD"/>
+<wire x1="55.88" y1="-53.34" x2="58.42" y2="-53.34" width="0.1524" layer="91"/>
+<wire x1="58.42" y1="-53.34" x2="58.42" y2="-66.04" width="0.1524" layer="91"/>
+<junction x="58.42" y="-66.04"/>
 </segment>
 <segment>
@@
 <pinref part="GND5" gate="G$1" pin="GND"/>
 <pinref part="C2" gate="G$1" pin="2"/>
+</segment>
+<segment>
+<pinref part="SW1" gate="G$1" pin="3"/>
+<wire x1="355.6" y1="12.7" x2="360.68" y2="12.7" width="0.1524" layer="91"/>
+<wire x1="360.68" y1="12.7" x2="360.68" y2="10.16" width="0.1524" layer="91"/>
+<pinref part="SW1" gate="G$1" pin="4"/>
+<wire x1="360.68" y1="10.16" x2="360.68" y2="7.62" width="0.1524" layer="91"/>
+<wire x1="355.6" y1="10.16" x2="360.68" y2="10.16" width="0.1524" layer="91"/>
+<junction x="360.68" y="10.16"/>
+<pinref part="GND1" gate="G$1" pin="GND"/>
+</segment>
+<segment>
+<pinref part="SW6" gate="G$1" pin="3"/>
+<wire x1="391.16" y1="12.7" x2="396.24" y2="12.7" width="0.1524" layer="91"/>
+<wire x1="396.24" y1="12.7" x2="396.24" y2="10.16" width="0.1524" layer="91"/>
+<pinref part="SW6" gate="G$1" pin="4"/>
+<wire x1="396.24" y1="10.16" x2="396.24" y2="7.62" width="0.1524" layer="91"/>
+<wire x1="391.16" y1="10.16" x2="396.24" y2="10.16" width="0.1524" layer="91"/>
+<junction x="396.24" y="10.16"/>
+<pinref part="GND3" gate="G$1" pin="GND"/>
 </segment>
 </net>
@@
 <segment>
 <pinref part="USB2" gate="G$1" pin="D-"/>
-<wire x1="55.88" y1="-58.42" x2="58.42" y2="-58.42" width="0.1524" layer="91"/>
-<label x="58.42" y="-58.42" size="1.27" layer="95" xref="yes"/>
+<wire x1="55.88" y1="-58.42" x2="60.96" y2="-58.42" width="0.1524" layer="91"/>
+<label x="60.96" y="-58.42" size="1.27" layer="95" xref="yes"/>
 </segment>
 </net>
@@
 <segment>
 <pinref part="USB2" gate="G$1" pin="D+"/>
-<wire x1="55.88" y1="-60.96" x2="58.42" y2="-60.96" width="0.1524" layer="91"/>
-<label x="58.42" y="-60.96" size="1.27" layer="95" xref="yes"/>
+<wire x1="55.88" y1="-60.96" x2="60.96" y2="-60.96" width="0.1524" layer="91"/>
+<label x="60.96" y="-60.96" size="1.27" layer="95" xref="yes"/>
 </segment>
 </net>
@@
 </segment>
 </net>
-<net name="VBATT" class="0">
-<segment>
-<wire x1="358.14" y1="-53.34" x2="355.6" y2="-53.34" width="0.1524" layer="91"/>
-<label x="355.6" y="-53.34" size="1.27" layer="95" rot="R180" xref="yes"/>
-<pinref part="U4" gate="G$1" pin="VBAT"/>
-</segment>
-</net>
+<net name="SW1" class="0">
+<segment>
+<pinref part="SW1" gate="G$1" pin="1"/>
+<wire x1="345.44" y1="12.7" x2="340.36" y2="12.7" width="0.1524" layer="91"/>
+<label x="340.36" y="12.7" size="1.27" layer="95" rot="R180" xref="yes"/>
+</segment>
+<segment>
+<pinref part="SW6" gate="G$1" pin="1"/>
+<wire x1="381" y1="12.7" x2="375.92" y2="12.7" width="0.1524" layer="91"/>
+<label x="375.92" y="12.7" size="1.27" layer="95" rot="R180" xref="yes"/>
+</segment>
+</net>

Commit message: changed schematic and board based on video take 002
Parts:
- added C22: 100n, LinnesLab-Passives:CAPACITOR0603
- added C23, C24: 47p, LinnesLab-Passives:CAPACITOR0603
- added JP2: (no value), LinnesLab-Switches:JUMPER-SMT_2_NO_SILK
- added LED5: RED, LinnesLab-LED:LED0603
- added LED6: YELLOW, LinnesLab-LED:LED0603
- added R1, R2: 0, LinnesLab-Passives:RESISTOR0603
- added R17, R18: 27, LinnesLab-Passives:RESISTOR0603
- added R19, R20: 1k, LinnesLab-Passives:RESISTOR0603
- added U5: FT231XS, LinnesLab-DigitalIC:FT231XS
Connections:
- new net !CTS: JP2.2, U5.!CTS
- new net FT3V3: U5.3V3OUT
- new net N$23: R17.2, U5.USBDM
- new net N$24: R18.2, U5.USBDP
- new net N$25: LED5.C, R19.2
- new net N$26: LED6.C, R20.2
- new net RXD.FT: R2.1
- new net RXD.NRF: R1.2, U2.P0.08
- new net RXLED: R19.1, U5.CBUS1
- new net TXD.FT: R1.1
- new net TXD.NRF: R2.2, U2.P0.06
- new net TXLED: R20.1, U5.CBUS2
- net 3.3V: now also C22.2, LED5.A, LED6.A, U5.!RESET, U5.VCCIO
- net DTR: now also U5.!DTR
- net GND: now also C22.1, C23.2, C24.1, JP2.1, U5.GND@16, U5.GND@6
- net RXD: now also U5.RXD; no longer U2.P0.08
- net SCL: now also R9.1; no longer R8.1
- net SDA: now also R8.1; no longer R9.1
- net TXD: now also U5.TXD; no longer U2.P0.06
- net USB+: now also C23.1, R18.1
- net USB-: now also C24.2, R17.1
- net V_USB: now also U5.VCC
Other:
- note added: "FTDI Serial-to-USB Converter"
- note added: "I don't remember if CTS needs to be grounded or left floating so here's a jumper to ground so it can be configued either way dynamically."
- note added: "Notes"
- note added: "TXD goes to RX on the other device RXD goes to TX on the other device"
- moved on the sheet: C10, C11, C12, C7, C8, C9, L2, LED3, LED4, R3, R4, R8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

Commit message: changes to top and bottom board based on take 002 video. Basic schematic and board is complete (no routing done yet)
Parts:
- renumbered SW6 to SW2
Connections:
- removed net BATT: R13.1, R14.2
- removed net CD1: SD2.CARD_DETECT
- removed net CHRG.STAT: CHRG2.STAT, R12.1
- removed net CS.OLED: U3./CS
- removed net DC.OLED: U3.DC/I2C_SA0
- removed net RESET.OLED: U3./RES
- removed net SD.CS: SD2.CS
- removed net SW1: SW1.1, SW2.1
- new net A4/BATT: R13.1, R14.2, U2.P0.28/AIN4
- new net A6/TIA: U2.P0.30/AIN6
- new net A7/PPG: U2.P0.31/AIN7
- new net D11/SW1: SW1.1, U2.P0.11
- new net D15/SW2: SW2.1, U2.P0.15
- new net D16/CS.OLED: U2.P0.16, U3./CS
- new net D27/CHRG.STATUS: CHRG2.STAT, R12.1, U2.P0.27
- new net D29/LED.CTRL: U2.P0.29/AIN5
- new net D3/RESET.OLED: U2.P0.04/AIN2, U3./RES
- new net D4/DC.OLED: U2.P0.03/AIN1, U3.DC/I2C_SA0
- new net D5/CD1: SD2.CARD_DETECT, U2.P0.05/AIN3
- new net D7/SD.CS: SD2.CS, U2.P0.07
Other:
- note added: "Digital Output"
